Commit message: ajout de la pince

File: robot_tennis/urdf/robot_tennis.urdf (robot description, URDF)
Before this commit: robot robot1, 4 links, 3 joints
Links:
- added link pince, mass 1; visual mesh filename=package://robot_tennis/meshs/pince2.dae
- link chassis: geometry collision box size=0.5 0.3 0.04; visual box size=0.5 0.3 0.04
Joints:
- added joint chassis_to_pince: type fixed, parent chassis, child pince, origin xyz=1 0 0 rpy=0 0 0, axis 0 0 0

Commit message: changement de pince

File: robot_tennis/urdf/robot_tennis.urdf (robot description, URDF)
Before this commit: robot robot1, 5 links, 4 joints
Links:
- removed link pince
- added link left_pince, mass 1; collision box size=0.4 0.03 0.08; visual box size=0.4 0.03 0.08
- added link right_pince, mass 1; collision box size=0.4 0.03 0.08; visual box size=0.4 0.03 0.08
Joints:
- removed joint chassis_to_pince
- added joint chassis_to_left_pince: type fixed, parent chassis, child left_pince, origin xyz=0.4 0.12 0.005 rpy=0 0.0 0.6, axis 0 1 0
- added joint chassis_to_right_pince: type fixed, parent chassis, child right_pince, origin xyz=0.4 -0.12 0.005 rpy=0 0.0 -0.6, axis 0 1 0

Commit message: modif

File: robot_tennis/urdf/robot_tennis.urdf (robot description, URDF)
Before this commit: robot robot1, 6 links, 5 joints
Links:
- link left_pince: mass 1 -> 0.2

Commit message: affichage pince

File: robot_tennis/urdf/robot_tennis.urdf (robot description, URDF)
Before this commit: robot robot1, 6 links, 5 joints
Links:
- removed link left_pince
- removed link right_pince
- added link pince, mass 0.2; collision mesh filename=package://robot_tennis/meshs/pince2.dae; visual mesh filename=package://robot_tennis/meshs/pince2.dae
Joints:
- removed joint chassis_to_left_pince
- removed joint chassis_to_right_pince
- added joint chassis_to_pince: type fixed, parent chassis, child pince, origin xyz=0.0 0 0.0 rpy=0 0 0, axis 0 0 0

Commit message: ajout Imu

File: robot_tennis/urdf/robot_tennis.urdf (robot description, URDF)
Before this commit: robot robot1, 5 links, 4 joints
Links:
- added link imu_link; visual cylinder length=0.02 radius=0.01
- link left_wheel: geometry collision cylinder length=0.03 radius=0.06; visual cylinder length=0.03 radius=0.06
- link right_wheel: geometry collision cylinder length=0.03 radius=0.06; visual cylinder length=0.03 radius=0.06
Joints:
- added joint chassis_to_imu: type fixed, parent chassis, child imu_link, origin xyz=0.17 0 0.07 rpy=0 0 0
- joint chassis_to_pince: origin xyz=0.0 0 0.0 rpy=0 0 0 -> xyz=0.0 0 0.05 rpy=0 0 0

Commit message: new pince

File: robot_tennis/urdf/robot_tennis.urdf (robot description, URDF)
Before this commit: robot robot1, 6 links, 5 joints
Links:
- link chassis: mass 1 -> 5
- link left_wheel: mass 1 -> 2
- link right_wheel: mass 1 -> 2
- link roue_folle: mass 1.0 -> 3.0
